File: ww-impedance-matching.sch (EAGLE design)
At the start: 80 parts, among them U4 ADG904BRUZ, X1 RASPI_BOARD_B+_E4P

Commit message: schematic done, basic component placement
Parts:
- removed TP1, TP2, TP3: TPTP14R, TestPoints:TPTP14R
- added C13: 1u, Capacitors:C-0603
- added C14: (no value), Capacitors:C-0805
- R_SCL, R_SDA: value (none) -> 10k
- renumbered JP_LDO_EN to JP.LDO.EN, JP_LDO_IN to JP.LDO.IN, JP_LDO_OUT to JP.LDO.OUT, U4 to MUX.RF.OUT
Connections:
- net N$1 renamed 5V.JMP
- net N$2 renamed 3V3.JMP
- net N$3 renamed SDA.IN
- net N$5 renamed SCL.IN
- net N$8 renamed LDO.OUT
- removed net N$13: TP1.TP, X1.GPIO04
- removed net N$14: TP2.TP, X1.GPIO25
- removed net N$16: TP3.TP, X1.GPIO24
- removed net N$7: JP.LDO.IN.1, U_LDO2.7.IN
- removed net VIN: C11.1, C12.1, C7.1, C9.1, MUX.RF.IN.VDD, MUX.RF.OUT.VDD, MUX.SCL.VDD, MUX.SDA.VDD
- new net LDO.IN: C13.1, JP.LDO.IN.1, U_LDO2.7.IN
- net 2.7V: now also C11.1, C12.1, C14.1, C7.1, C9.1, MUX.RF.IN.VDD, MUX.RF.OUT.VDD, MUX.SCL.VDD, MUX.SDA.VDD
- net GND: now also C13.2, C14.2
Other:
- note added: "Input signal should be less than 2.7V pk-pk This is due to the SP4T mux's voltage range."

Commit message: filter placement
Connections:
- net N$29 renamed RF.F1.0
- net N$39 renamed RF.F3.0
- net N$4 renamed RF.F0.0
- net N$49 renamed RF.F2.0
Changed lines of the file:
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@@
 <class number="1" name="PWR" width="0.3048" drill="0">
+</class>
+<class number="2" name="RF" width="0" drill="0">
 </class>
 </classes>
@@
 </segment>
 </net>
-<net name="N$4" class="0">
+<net name="RF.F0.0" class="2">
 <segment>
 <pinref part="CT.F0.1" gate="G$1" pin="C+"/>
@@
 </segment>
 </net>
-<net name="F0.OUT" class="0">
+<net name="F0.OUT" class="2">
 <segment>
 <pinref part="Z.F0.3" gate="G$1" pin="1"/>
@@
 </segment>
 </net>
-<net name="F0.IN" class="0">
+<net name="F0.IN" class="2">
 <segment>
 <pinref part="CT.F0.0" gate="G$1" pin="C+"/>
@@
 </segment>
 </net>
-<net name="N$29" class="0">
+<net name="RF.F1.0" class="2">
 <segment>
 <pinref part="CT.F1.1" gate="G$1" pin="C+"/>
@@
 </segment>
 </net>
-<net name="F2.IN" class="0">
+<net name="F2.IN" class="2">
 <segment>
 <pinref part="CT.F2.0" gate="G$1" pin="C+"/>
@@
 </segment>
 </net>
-<net name="F1.IN" class="0">
+<net name="F1.IN" class="2">
 <segment>
 <pinref part="CT.F1.0" gate="G$1" pin="C+"/>
@@
 </segment>
 </net>
-<net name="N$49" class="0">
+<net name="RF.F2.0" class="2">
 <segment>
 <pinref part="CT.F2.1" gate="G$1" pin="C+"/>
@@
 </segment>
 </net>
-<net name="F2.OUT" class="0">
+<net name="F2.OUT" class="2">
 <segment>
 <pinref part="Z.F2.3" gate="G$1" pin="1"/>
@@
 </segment>
 </net>
-<net name="N$39" class="0">
+<net name="RF.F3.0" class="2">
 <segment>
 <pinref part="CT.F3.1" gate="G$1" pin="C+"/>
@@
 </segment>
 </net>
-<net name="F3.OUT" class="0">
+<net name="F3.OUT" class="2">
 <segment>
 <pinref part="Z.F3.3" gate="G$1" pin="1"/>
@@
 </segment>
 </net>
-<net name="F3.IN" class="0">
+<net name="F3.IN" class="2">
 <segment>
 <pinref part="CT.F3.0" gate="G$1" pin="C+"/>
@@
 </segment>
 </net>
-<net name="RF_OUT" class="0">
+<net name="RF_OUT" class="2">
 <segment>
 <pinref part="MUX.RF.OUT" gate="A" pin="RFC"/>
@@
 </segment>
 </net>
-<net name="RF_IN" class="0">
+<net name="RF_IN" class="2">
 <segment>
 <pinref part="SMA.IN" gate="G1" pin="1"/>
@@
 </segment>
 </net>
-<net name="F1.OUT" class="0">
+<net name="F1.OUT" class="2">
 <segment>
 <pinref part="Z.F1.2" gate="G$1" pin="1"/>

Commit message: mostly routed
Parts:
- renumbered JP.F0.SD0 to JP.F0.SDA0, JP.F1.SD0 to JP.F1.SDA0, JP.F2.SD0 to JP.F2.SDA0, JP.F3.SD0 to JP.F3.SDA0
Connections:
- net N$11: now also X1.GPIO27; no longer X1.GPIO18
Other:
- moved on the sheet: MUX0, MUX1, R2, R3, R4, T.M0, T.M1

Commit message: add BOM
Parts:
- X1: MP (none) -> TSM-110-02-S-DV; MPN (none) -> TSM-110-02-S-DV; PART_NO (none) -> TSM-110-02-S-DV
Changed lines of the file:
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@@
 </classes>
 <parts>
-<part name="X1" library="raspberrypi_bastelstube_v13" deviceset="RASPI_BOARD_B+" device="_E4P"/>
+<part name="X1" library="raspberrypi_bastelstube_v13" deviceset="RASPI_BOARD_B+" device="_E4P">
+<attribute name="MP" value="TSM-110-02-S-DV"/>
+<attribute name="MPN" value="TSM-110-02-S-DV"/>
+<attribute name="PART_NO" value="TSM-110-02-S-DV"/>
+</part>
 <part name="GND1" library="Supplies" deviceset="GND" device=""/>
 <part name="+3V1" library="Supplies" deviceset="+3V3" device=""/>
@@
 </plain>
 <instances>
-<instance part="X1" gate="G$1" x="88.9" y="101.6" smashed="yes" rot="MR0"/>
+<instance part="X1" gate="G$1" x="88.9" y="101.6" smashed="yes" rot="MR0">
+<attribute name="MP" x="88.9" y="101.6" size="1.778" layer="96" rot="MR0" display="off"/>
+<attribute name="PART_NO" x="88.9" y="101.6" size="1.778" layer="96" rot="MR0" display="off"/>
+<attribute name="MPN" x="88.9" y="101.6" size="1.778" layer="96" rot="MR0" display="off"/>
+</instance>
 <instance part="GND1" gate="1" x="88.9" y="55.88" smashed="yes" rot="MR0">
 <attribute name="VALUE" x="91.44" y="53.34" size="1.778" layer="96" rot="MR0"/>

Commit message: revA production
Parts:
- added LOGO1: LOGO-CMU, Graphics:LOGO-CMU
Changed lines of the file:
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@@
 <attribute name="PART_NO" value="CC0805KPX5R6BB106"/>
 </part>
+<part name="LOGO1" library="Graphics" deviceset="LOGO-CMU" device=""/>
 </parts>
 <sheets>
@@
 <attribute name="MP" x="210.82" y="378.46" size="1.778" layer="96" display="off"/>
 </instance>
+<instance part="LOGO1" gate="G$1" x="541.02" y="45.72" smashed="yes"/>
 </instances>
 <busses>
@@
 <segment>
 <wire x1="147.32" y1="287.02" x2="147.32" y2="10.16" width="0.762" layer="92"/>
-<wire x1="147.32" y1="10.16" x2="419.1" y2="12.7" width="0.762" layer="92"/>
-<wire x1="419.1" y1="12.7" x2="419.1" y2="218.44" width="0.762" layer="92"/>
+<wire x1="147.32" y1="10.16" x2="419.1" y2="10.16" width="0.762" layer="92"/>
+<wire x1="419.1" y1="10.16" x2="419.1" y2="215.9" width="0.762" layer="92"/>
 <label x="393.7" y="17.78" size="2.54" layer="95"/>
 <label x="152.4" y="170.18" size="2.54" layer="95"/>
